File: AOI_Hutschiene.brd (EAGLE design)
At the start: 99.1 x 85.7 mm, 33 parts, among them IC1 l4940, SW1 EC12E_SW

Commit message: updated design
Parts:
- removed H5, H6, H7: MOUNT-PAD-ROUND3.2, holes:3,2-PAD
- removed SV3: (no value), con-lsta:FE05W
- added D1: 1N4148DO35-7, diode:DO35-7
- added R5, R6: 4k7, resistor:0207/2V
- added R7, R8: 22k, resistor:0207/10
- added SV5: (no value), con-lstb:MA04-1
- C3: value 1000uF -> 1mF
- F2: value FUSESH22,5 -> 100mA_or_smaller
- R1, R2: value (none) -> 180
- TR1: value 6v -> 6V, 300mA
- moved SV2 30.1 mm to (62.9, 34.9), turned to 90 degrees
- moved SG1 14.4 mm to (95.3, 26.9), turned to 90 degrees
- moved LED_MIX 8.89 mm to (92.7, 54.0)
- moved S1_MIX 8.89 mm to (92.7, 41.9)
- moved R1 8.47 mm to (87.0, 48.9)
- moved SW1 4.45 mm to (81.9, 17.1)
- moved C4 2.54 mm to (10.8, 71.1)
- moved R2 2.01 mm to (76.8, 48.9)
- moved R3 1.27 mm to (19.7, 62.2)
- moved R4 1.27 mm to (19.7, 59.7)
- moved SV4 0.63 mm to (27.3, 73.7)
Connections:
- net N$12 renamed DSS_VCC
- removed net REL_HEAT_2: U$1.A1
- removed net REL_MIX_2: U$1.A3
- net DISP_CLK_IN: now also SV5.4; no longer SV3.4
- net DISP_DATA_IN: now also SV5.3; no longer SV3.3
- net GND: now also IC2.3, IC2.4, IC2.5, IC2.6, IC2.7, IC2.8, R7.1, R8.1
- net GNDIO: now also SV5.1; no longer SV3.1
- net N$1: now also R5.2, R6.2
- net N$2: now also R5.1
- net N$3: now also R6.1
- net REL_HEAT_OUT: now also D1.A, R8.2
- net REL_MIX_OUT: now also D1.C, R7.2
- net VCCIO: now also SV5.2; no longer SV3.2
Routing:
- net BUZ_IN: track 6.50 -> 45.1 mm, vias 0 -> 1
- net GNDIO: track 46.1 -> 9.42 mm, vias 5 -> 25
- net REL_HEAT_OUT_2: track 39.0 -> 13.8 mm
- net REL_HEAT_IN: track 33.8 -> 12.0 mm
- net DISP_CLK_IN: track 41.7 -> 20.9 mm, vias 1 -> 0
- net ENC_SW_IN: track 14.8 -> 33.7 mm, vias 0 -> 2
- net ENC_R_IN: track 26.8 -> 44.2 mm
- net DISP_DATA_IN: track 43.4 -> 26.3 mm, vias 1 -> 0
- net AUX_IO: track 17.0 -> 0.00 mm, vias 1 -> 0
- net REL_MIX_OUT_2: track 20.0 -> 35.2 mm
- net REL_MIX_IN: track 15.3 -> 29.9 mm
- net N$1: track 45.1 -> 56.5 mm
- net REL_MIX_OUT: track 39.8 -> 50.6 mm
- net N$3: track 11.9 -> 21.5 mm
- net N$2: track 20.9 -> 30.0 mm
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Other:
- board size 99.1 x 85.7 mm -> 99.1 x 101 mm
- board text added: "Auto"
- board text added: "LCD"
- board text added: "Man_ON"
- board text added: "OFF"
- board text added: "v cut"

Commit message: Bugfixes to schematic and board (D1, R3/R4)
- D1: Wrong position. Declared as "dont use"
- R3/R4: Wrong silk screen position in PCB. Fixed by interchanging component names in schematic
Parts:
- B1: value (none) -> B40C2000
- IC2: value (none) -> ULN2803
- LED_HEAT: value (none) -> LED_HEAT_RED
- LED_MIX: value (none) -> LED_MIX_YEL
- R1, R2: value 180 -> 120
- R3: value 12 -> 4k7
- R4: value 4k7 -> 20
- U$1: value NANO -> ArdNano_with_socket
- moved R3 2.54 mm to (19.7, 59.7), turned to 0 degrees
- moved R4 2.54 mm to (19.7, 62.2), turned to 180 degrees
Connections:
- removed net DSS_VCC: C4.2, R3.1, X2.4
- new net N$12: C4.2, R4.1, X2.4
- net DSS_DATA: now also R3.2; no longer R4.2
- net VCC: now also R3.1, R4.2; no longer R3.2, R4.1
Routing:
- net N$12: track 0.00 -> 31.5 mm
- net DSS_VCC: track 31.5 -> 0.00 mm
Other:
- board text added: "HEAT"
- board text added: "MIX"
- board text added: "REL_+"
- board text added: "SENS_DATA"
- board text added: "SENS_GND"
- board text added: "SENS_VCC"
- board text added: "arduino: with socket, top side"
- board text removed: "Auto"
- board text removed: "Man_ON"
- board text removed: "OFF"
